Commit message: make to match our robot

File: description/gazebo_control.xacro (robot description, xacro)
@@ -1,4 +1,5 @@
 <?xml version="1.0"?>
 <robot xmlns:xacro="http://www.ros.org/wiki/xacro">
+	<!-- holonomic control gazebo -->
 	<gazebo>
 		<plugin name="holonomic_control" filename="libgazebo_ros_planar_move.so">
@@ -10,4 +11,4 @@
 			<publishTF>true</publishTF>
     	</plugin>
-  </gazebo>
+  	</gazebo>
 </robot>

File: description/robot.urdf.xacro (robot description, xacro)
@@ -1,6 +1,6 @@
 <?xml version="1.0"?>
 <robot xmlns:xacro="http://www.ros.org/wiki/xacro"  name="robot">
-	<xacro:include filename="robot_core_highres.xacro"/>
-    <!--<xacro:include filename="robot_core.xacro"/>--> <!--Uncomment to use low res mode-->
+	<!-- <xacro:include filename="robot_core_highres.xacro"/> -->
+    <xacro:include filename="robot_core.xacro"/> <!--Uncomment to use low res mode-->
     <xacro:include filename="gazebo_control.xacro"/>
 </robot>

File: description/robot_core.xacro (robot description, xacro)
@@ -3,11 +3,5 @@
     <xacro:include filename="inertial_macros.xacro"/>
     <material name="white">
-        <color rgba="1 1 1 1"/>
-    </material>
-    <material name="orange">
-		<color rgba="1 0.3 0.1 1"/>
-    </material>
-    <material name="blue">
-		<color rgba="0.2 0.2 1 1"/>
+        <color rgba="0.5 0.5 0.5 1"/>
     </material>
     <material name="black">
@@ -17,36 +11,209 @@
     <link name="base_link">
     </link>
-    <!-- CHASSIS LINK -->
-	<joint name="chassis_joint" type="fixed">
-		<parent link="base_link"/>
-		<child link="chassis"/>
-		<origin xyz="0 0 0"/>
-	</joint>
-	<link name="chassis">
-		<visual>
-			<origin xyz="0 0 0.1"/>
-			<geometry>
-				<box size="0.5 0.5 0.03"/>
-			</geometry>
-			<material name="white"/>
-		</visual>
-		<collision>
-			<origin xyz="0 0 0.1"/>
-			<geometry>
-				<box size="0.5 0.5 0.03"/>
-			</geometry>
-		</collision>
-		<xacro:inertial_box mass="0.2" x="0.5" y="0.5" z="0.03">
-        	<origin xyz="0 0 0.1" rpy="0 0 0"/>
-    	</xacro:inertial_box>
-	</link>
-	<gazebo reference="chassis">
-        <material>Gazebo/White</material>
-    </gazebo>
+	<!-- left ft slot -->
+	<joint name="left_ft_joint" type="fixed">
+		<parent link="base_link"/>
+		<child link="left_ft_link"/>
+		<origin xyz="0.185 0.225 0.134" rpy="${pi/2} 0 0"/>
+		<axis xyz="0 0 1"/>
+	</joint>
+	<link name="left_ft_link">
+		<visual>
+			<origin xyz="0 0 0.1"/>
+			<geometry>
+				<mesh filename="package://holonomic/meshes/2020_AL-Profile.stl" scale="0.001 0.001 0.025"/>
+			</geometry>
+			<material name="white"/>
+		</visual>
+		<collision>
+			<origin xyz="0 0 0.1"/>
+			<geometry>
+				<box size="0.0 0.0 0.0"/>
+			</geometry>
+		</collision>
+		<xacro:inertial_box mass="0.2" x="0.5" y="0.5" z="0.03">
+        	<origin xyz="0 0 0.1" rpy="0 0 0"/>
+    	</xacro:inertial_box>
+	</link>
+	<!-- left bt slot -->
+	<joint name="left_bt_joint" type="fixed">
+		<parent link="base_link"/>
+		<child link="left_bt_link"/>
+		<origin xyz="-0.205 0.225 0.134" rpy="${pi/2} 0 0"/>
+		<axis xyz="0 0 1"/>
+	</joint>
+	<link name="left_bt_link">
+		<visual>
+			<origin xyz="0 0 0.1"/>
+			<geometry>
+				<mesh filename="package://holonomic/meshes/2020_AL-Profile.stl" scale="0.001 0.001 0.025"/>
+			</geometry>
+			<material name="white"/>
+		</visual>
+		<collision>
+			<origin xyz="0 0 0.1"/>
+			<geometry>
+				<box size="0.0 0.0 0.0"/>
+			</geometry>
+		</collision>
+		<xacro:inertial_box mass="0.2" x="0.5" y="0.5" z="0.03">
+        	<origin xyz="0 0 0.1" rpy="0 0 0"/>
+    	</xacro:inertial_box>
+	</link>
+	<!-- left ll slot -->
+	<joint name="left_ll_joint" type="fixed">
+		<parent link="base_link"/>
+		<child link="left_ll_link"/>
+		<origin xyz="-0.3 0.105 0.15" rpy="0 ${pi/2}  0"/>
+		<axis xyz="0 0 1"/>
+	</joint>
+	<link name="left_ll_link">
+		<visual>
+			<origin xyz="0 0 0.1"/>
+			<geometry>
+				<mesh filename="package://holonomic/meshes/2020_AL-Profile.stl" scale="0.001 0.001 0.04"/>
+			</geometry>
+			<material name="white"/>
+		</visual>
+		<collision>
+			<origin xyz="0 0 0.1"/>
+			<geometry>
+				<box size="0.0 0.0 0.0"/>
+			</geometry>
+		</collision>
+		<xacro:inertial_box mass="0.2" x="0.5" y="0.5" z="0.03">
+        	<origin xyz="0 0 0.1" rpy="0 0 0"/>
+    	</xacro:inertial_box>
+	</link>
+	<!-- left lr slot -->
+	<joint name="left_lr_joint" type="fixed">
+		<parent link="base_link"/>
+		<child link="left_lr_link"/>
+		<origin xyz="-0.3 -0.125 0.15" rpy="0 ${pi/2}  0"/>
+		<axis xyz="0 0 1"/>
+	</joint>
+	<link name="left_lr_link">
+		<visual>
+			<origin xyz="0 0 0.1"/>
+			<geometry>
+				<mesh filename="package://holonomic/meshes/2020_AL-Profile.stl" scale="0.001 0.001 0.04"/>
+			</geometry>
+			<material name="white"/>
+		</visual>
+		<collision>
+			<origin xyz="0 0 0.1"/>
+			<geometry>
+				<box size="0.0 0.0 0.0"/>
+			</geometry>
+		</collision>
+		<xacro:inertial_box mass="0.2" x="0.5" y="0.5" z="0.03">
+        	<origin xyz="0 0 0.1" rpy="0 0 0"/>
+    	</xacro:inertial_box>
+	</link>
+	<!-- servo fr -->
+	<joint name="servo_fr_joint" type="fixed">
+		<parent link="base_link"/>
+		<child link="servo_fr_link"/>
+		<origin xyz="0.19717 0.0 0.1" rpy="${pi/2} ${-pi/2} 0"/>
+		<axis xyz="0 0 1"/>
+	</joint>
+	<link name="servo_fr_link">
+		<visual>
+			<origin xyz="0 0 0.1"/>
+			<geometry>
+				<mesh filename="package://holonomic/meshes/servomotor.stl" scale="0.0030 0.0030 0.0026"/>
+			</geometry>
+			<material name="white"/>
+		</visual>
+		<collision>
+			<origin xyz="0 0 0.1"/>
+			<geometry>
+				<box size="0.0 0.0 0.0"/>
+			</geometry>
+		</collision>
+		<xacro:inertial_box mass="0.2" x="0.5" y="0.5" z="0.03">
+        	<origin xyz="0 0 0.1" rpy="0 0 0"/>
+    	</xacro:inertial_box>
+	</link>
+	<!-- servo br -->
+	<joint name="servo_br_joint" type="fixed">
+		<parent link="base_link"/>
+		<child link="servo_br_link"/>
+		<origin xyz="-0.19717 0.0 0.1" rpy="${pi/2} ${-pi/2} 0"/>
+		<axis xyz="0 0 1"/>
+	</joint>
+	<link name="servo_br_link">
+		<visual>
+			<origin xyz="0 0 0.1"/>
+			<geometry>
+				<mesh filename="package://holonomic/meshes/servomotor.stl" scale="0.0030 0.0030 0.0026"/>
+			</geometry>
+			<material name="white"/>
+		</visual>
+		<collision>
+			<origin xyz="0 0 0.1"/>
+			<geometry>
+				<box size="0.0 0.0 0.0"/>
+			</geometry>
+		</collision>
+		<xacro:inertial_box mass="0.2" x="0.5" y="0.5" z="0.03">
+        	<origin xyz="0 0 0.1" rpy="0 0 0"/>
+    	</xacro:inertial_box>
+	</link>
+	<!-- servo bl -->
+	<joint name="servo_bl_joint" type="fixed">
+		<parent link="base_link"/>
+		<child link="servo_bl_link"/>
+		<origin xyz="-0.19717 0.0 0.1" rpy="${-pi/2} ${-pi/2} 0"/>
+		<axis xyz="0 0 1"/>
+	</joint>
+	<link name="servo_bl_link">
+		<visual>
+			<origin xyz="0 0 0.1"/>
+			<geometry>
+				<mesh filename="package://holonomic/meshes/servomotor.stl" scale="0.0030 0.0030 0.0026"/>
+			</geometry>
+			<material name="white"/>
+		</visual>
+		<collision>
+			<origin xyz="0 0 0.1"/>
+			<geometry>
+				<box size="0.0 0.0 0.0"/>
+			</geometry>
+		</collision>
+		<xacro:inertial_box mass="0.2" x="0.5" y="0.5" z="0.03">
+        	<origin xyz="0 0 0.1" rpy="0 0 0"/>
+    	</xacro:inertial_box>
+	</link>
+	<!-- servo fl -->
+	<joint name="servo_fl_joint" type="fixed">
+		<parent link="base_link"/>
+		<child link="servo_fl_link"/>
+		<origin xyz="0.19717 0.0 0.1" rpy="${-pi/2} ${-pi/2} 0"/>
+		<axis xyz="0 0 1"/>
+	</joint>
+	<link name="servo_fl_link">
+		<visual>
+			<origin xyz="0 0 0.1"/>
+			<geometry>
+				<mesh filename="package://holonomic/meshes/servomotor.stl" scale="0.0030 0.0030 0.0026"/>
+			</geometry>
+			<material name="white"/>
+		</visual>
+		<collision>
+			<origin xyz="0 0 0.1"/>
+			<geometry>
+				<box size="0.0 0.0 0.0"/>
+			</geometry>
+		</collision>
+		<xacro:inertial_box mass="0.2" x="0.5" y="0.5" z="0.03">
+        	<origin xyz="0 0 0.1" rpy="0 0 0"/>
+    	</xacro:inertial_box>
+	</link>
 	<!-- WHEEL1 LINK -->
 	<joint name="wheel1_joint" type="continuous">
 		<parent link="base_link"/>
 		<child link="wheel1_link"/>
-		<origin xyz="0 0.27 0.08" rpy="-${pi/2} 0 0"/>
+		<origin xyz="0.19717 -0.20 0.08" rpy="${-pi/2} ${-pi/2} 0"/>
 		<axis xyz="0 0 1"/>
 	</joint>
@@ -54,5 +221,5 @@
 		<visual>
 			<geometry>
-				<cylinder radius="0.08" length="0.04"/>
+				<mesh filename="package://holonomic/meshes/wheel.stl" scale="0.00172 0.00172 0.00095"/>
 			</geometry>
 		</visual>
@@ -67,5 +234,5 @@
 	</link>
 	<gazebo reference="wheel1_link">
-        <material>Gazebo/Black</material>
+        <material>Gazebo/White</material>
 		<mu1 value="0.5"/>
 		<mu2 value="0.5"/>
@@ -75,5 +242,5 @@
 		<parent link="base_link"/>
 		<child link="wheel2_link"/>
-		<origin xyz="0 -0.27 0.08" rpy="${pi/2} 0 0"/>
+		<origin xyz="-0.19717 -0.20 0.08" rpy="${-pi/2} ${-pi/2} 0"/>
 		<axis xyz="0 0 -1"/>
 	</joint>
@@ -81,5 +248,5 @@
 		<visual>
 			<geometry>
-				<cylinder radius="0.08" length="0.04"/>
+				<mesh filename="package://holonomic/meshes/wheel.stl" scale="0.00172 0.00172 0.00095"/>
 			</geometry>
 		</visual>
@@ -94,5 +261,5 @@
 	</link>
 	<gazebo reference="wheel2_link">
-        <material>Gazebo/Black</material>
+        <material>Gazebo/White</material>
 		<mu1 value="0.5"/>
 		<mu2 value="0.5"/>
@@ -102,5 +269,5 @@
 		<parent link="base_link"/>
 		<child link="wheel3_link"/>
-		<origin xyz="0.27 0 0.08" rpy="${-pi/2} 0 ${-pi/2}"/>
+		<origin xyz="0.19717 0.20 0.08" rpy="${pi/2} ${-pi/2} 0"/>
 		<axis xyz="0 0 1"/>
 	</joint>
@@ -108,5 +275,5 @@
 		<visual>
 			<geometry>
-				<cylinder radius="0.08" length="0.04"/>
+				<mesh filename="package://holonomic/meshes/wheel.stl" scale="0.00172 0.00172 0.00095"/>
 			</geometry>
 		</visual>
@@ -121,5 +288,5 @@
 	</link>
 	<gazebo reference="wheel3_link">
-        <material>Gazebo/Black</material>
+        <material>Gazebo/White</material>
 		<mu1 value="0.5"/>
 		<mu2 value="0.5"/>
@@ -129,5 +296,5 @@
 		<parent link="base_link"/>
 		<child link="wheel4_link"/>
-		<origin xyz="-0.27 0 0.08" rpy="${pi/2} 0 ${-pi/2}"/>
+		<origin xyz="-0.19717 0.20 0.08" rpy="${pi/2} ${-pi/2} 0"/>
 		<axis xyz="0 0 -1"/>
 	</joint>
@@ -135,5 +302,5 @@
 		<visual>
 			<geometry>
-				<cylinder radius="0.08" length="0.04"/>
+				<mesh filename="package://holonomic/meshes/wheel.stl" scale="0.00172 0.00172 0.00095"/>
 			</geometry>
 		</visual>
@@ -148,5 +315,5 @@
 	</link>
 	<gazebo reference="wheel4_link">
-        <material>Gazebo/Black</material>
+        <material>Gazebo/White</material>
 		<mu1 value="0.5"/>
 		<mu2 value="0.5"/>

Commit message: both cameras on

File: description/gazebo_control.xacro (robot description, xacro)
@@ -1,4 +1,83 @@
 <?xml version="1.0"?>
 <robot xmlns:xacro="http://www.ros.org/wiki/xacro">
+	<!-- cameras  -->
+	<gazebo reference='cam_1_link'>
+		<sensor type="camera" name="cam_1_link">
+		<update_rate>30.0</update_rate>
+		<camera name="cam_1_link">
+			<horizontal_fov>1.3962634</horizontal_fov>
+			<image>
+			<width>800</width>
+			<height>800</height>
+			<format>R8G8B8</format>
+			</image>
+			<clip>
+			<near>0.02</near>
+			<far>300</far>
+			</clip>
+			<noise>
+			<type>gaussian</type>
+			<!-- Noise is sampled independently per pixel on each frame.
+				That pixel's noise value is added to each of its color
+				channels, which at that point lie in the range [0,1]. -->
+			<mean>0.0</mean>
+			<stddev>0.007</stddev>
+			</noise>
+		</camera>
+		<plugin name="camera_1_controller" filename="libgazebo_ros_camera.so">
+			<alwaysOn>true</alwaysOn>
+			<updateRate>0.0</updateRate>
+			<cameraName>cam_1_link</cameraName>
+			<imageTopicName>image_raw</imageTopicName>
+			<cameraInfoTopicName>camera_info</cameraInfoTopicName>
+			<frameName>uoz_bot/camera_1</frameName>
+			<hackBaseline>0.07</hackBaseline>
+			<distortionK1>0.0</distortionK1>
+			<distortionK2>0.0</distortionK2>
+			<distortionK3>0.0</distortionK3>
+			<distortionT1>0.0</distortionT1>
+			<distortionT2>0.0</distortionT2>
+		</plugin>
+		</sensor>
+	</gazebo>
+	<gazebo reference='cam_2_link'>
+		<sensor type="camera" name="cam_2_link">
+		<update_rate>30.0</update_rate>
+		<camera name="cam_2_link">
+			<horizontal_fov>1.3962634</horizontal_fov>
+			<image>
+			<width>800</width>
+			<height>800</height>
+			<format>R8G8B8</format>
+			</image>
+			<clip>
+			<near>0.02</near>
+			<far>300</far>
+			</clip>
+			<noise>
+			<type>gaussian</type>
+			<!-- Noise is sampled independently per pixel on each frame.
+				That pixel's noise value is added to each of its color
+				channels, which at that point lie in the range [0,1]. -->
+			<mean>0.0</mean>
+			<stddev>0.007</stddev>
+			</noise>
+		</camera>
+		<plugin name="camera_2_controller" filename="libgazebo_ros_camera.so">
+			<alwaysOn>true</alwaysOn>
+			<updateRate>0.0</updateRate>
+			<cameraName>cam_2_link</cameraName>
+			<imageTopicName>image_raw</imageTopicName>
+			<cameraInfoTopicName>camera_info</cameraInfoTopicName>
+			<frameName>uoz_bot/camera_2</frameName>
+			<hackBaseline>0.07</hackBaseline>
+			<distortionK1>0.0</distortionK1>
+			<distortionK2>0.0</distortionK2>
+			<distortionK3>0.0</distortionK3>
+			<distortionT1>0.0</distortionT1>
+			<distortionT2>0.0</distortionT2>
+		</plugin>
+		</sensor>
+	</gazebo>
 	<!-- holonomic control gazebo -->
 	<gazebo>

File: description/robot_core.xacro (robot description, xacro)
@@ -319,3 +319,124 @@
 		<mu2 value="0.5"/>
     </gazebo>
+	<joint name="cam_ftt_joint" type="fixed">
+		<parent link="base_link"/>
+		<child link="cam_ftt_link"/>
+		<origin xyz="0.088 0.21 0.35" rpy="${pi/2} ${-pi/2} 0"/>
+		<axis xyz="0 0 -1"/>
+	</joint>
+	<link name="cam_ftt_link">
+		<visual>
+			<origin xyz="0 0 0.1"/>
+			<geometry>
+				<mesh filename="package://holonomic/meshes/2020_AL-Profile.stl" scale="0.001 0.001 0.022"/>
+				<!-- <box size="0.01 0.01 0.77"/> -->
+			</geometry>
+			<material name="white"/>
+		</visual>
+		<collision>
+			<origin xyz="0 0 0.1"/>
+			<geometry>
+				<box size="0.0 0.0 0.0"/>
+			</geometry>
+		</collision>
+		<xacro:inertial_box mass="0.2" x="0.5" y="0.5" z="0.03">
+        	<origin xyz="0 0 0.1" rpy="0 0 0"/>
+    	</xacro:inertial_box>
+	</link>
+	<joint name="cam_1_joint" type="fixed">
+		<parent link="base_link"/>
+		<child link="cam_1_link"/>
+		<origin xyz="0.076 -0.07 0.24" rpy="0 0 0"/>
+		<axis xyz="0 0 -1"/>
+	</joint>
+	<link name="cam_1_link">
+		<visual>
+			<origin xyz="0 0 0.1" rpy="0 0.15 0"/>
+			<geometry>
+				<box size="0.03 0.03 0.03"/>
+			</geometry>
+			<material name="white"/>
+		</visual>
+		<collision>
+			<origin xyz="0 0 0.1"/>
+			<geometry>
+				<box size="0.0 0.0 0.0"/>
+			</geometry>
+		</collision>
+		<xacro:inertial_box mass="0.2" x="0.5" y="0.5" z="0.03">
+        	<origin xyz="0 0 0.1" rpy="0 0 0"/>
+    	</xacro:inertial_box>
+	</link>
+	<joint name="cam_2_joint" type="fixed">
+		<parent link="base_link"/>
+		<child link="cam_2_link"/>
+		<origin xyz="0.076 0.07 0.24" rpy="0 0 0"/>
+		<axis xyz="0 0 -10"/>
+	</joint>
+	<link name="cam_2_link">
+		<visual>
+			<origin xyz="0 0 0.1" rpy="0 0.50 0"/>
+			<geometry>
+				<box size="0.03 0.03 0.03"/>
+			</geometry>
+			<material name="white"/>
+		</visual>
+		<collision>
+			<origin xyz="0 0 0.1"/>
+			<geometry>
+				<box size="0.0 0.0 0.0"/>
+			</geometry>
+		</collision>
+		<xacro:inertial_box mass="0.2" x="0.5" y="0.5" z="0.03">
+        	<origin xyz="0 0 0.1" rpy="0 0 0"/>
+    	</xacro:inertial_box>
+	</link>
+	<joint name="cam_pole_1_link_joint" type="fixed">
+		<parent link="base_link"/>
+		<child link="cam_pole_1_link"/>
+		<origin xyz="0.07 0.105 0.03" rpy="0 0 0"/>
+		<axis xyz="0 0 -1"/>
+	</joint>
+	<link name="cam_pole_1_link">
+		<visual>
+			<origin xyz="0 0 0.1"/>
+			<geometry>
+				<mesh filename="package://holonomic/meshes/2020_AL-Profile.stl" scale="0.001 0.001 0.025"/>
+			</geometry>
+			<material name="white"/>
+		</visual>
+		<collision>
+			<origin xyz="0 0 0.1"/>
+			<geometry>
+				<box size="0.0 0.0 0.0"/>
+			</geometry>
+		</collision>
+		<xacro:inertial_box mass="0.2" x="0.5" y="0.5" z="0.03">
+        	<origin xyz="0 0 0.1" rpy="0 0 0"/>
+    	</xacro:inertial_box>
+	</link>
+	<joint name="cam_pole_2_link_joint" type="fixed">
+		<parent link="base_link"/>
+		<child link="cam_pole_2_link"/>
+		<origin xyz="0.07 -0.125 0.03" rpy="0 0 0"/>
+		<axis xyz="0 0 -1"/>
+	</joint>
+	<link name="cam_pole_2_link">
+		<visual>
+			<origin xyz="0 0 0.1"/>
+			<geometry>
+				<mesh filename="package://holonomic/meshes/2020_AL-Profile.stl" scale="0.001 0.001 0.025"/>
+			</geometry>
+			<material name="white"/>
+		</visual>
+		<collision>
+			<origin xyz="0 0 0.1"/>
+			<geometry>
+				<box size="0.0 0.0 0.0"/>
+			</geometry>
+		</collision>
+		<xacro:inertial_box mass="0.2" x="0.5" y="0.5" z="0.03">
+        	<origin xyz="0 0 0.1" rpy="0 0 0"/>
+    	</xacro:inertial_box>
+	</link>
 </robot>
